File: HF1R00/Design/HF1R01.brd (EAGLE design)
At the start: 34.6 x 90 mm, 18 parts, among them P1 HEXABIT_17.32_TWO_SIDES, P2 HEXABIT_17.32_TWO_SIDES, P3 HEXABIT_17.32_TWO_SIDES, P4 HEXABIT_17.32_TWO_SIDES, P5 HEXABIT_17.32_TWO_SIDES, P6 HEXABIT_17.32_TWO_SIDES, U1 CAT24C32WI-GT3

Commit message: - Added a header pin to isolate the 3.3v between ras and modules.. - Changed to Rev1.. - Updated BOM and Document..
Parts:
- added JP4: 61300211121, jumper:JP1
Connections:
- new net N$3: C2.1, JP4.1, SV1.1, SV1.17
- net +3V3: now also JP4.2; no longer C2.1, SV1.1, SV1.17
Routing:
- net N$3: track 0.00 -> 34.1 mm
- net +3V3: track 14.5 -> 5.13 mm
- net TXD3: track 26.3 -> 27.6 mm
Other:
- board text added: "HF1R01"
- board text removed: "HF1R00"
Changed lines of the file:
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@@
 <?xml version="1.0" encoding="utf-8"?>
 <!DOCTYPE eagle SYSTEM "eagle.dtd">
-<eagle version="9.3.0">
+<eagle version="9.6.2">
 <drawing>
 <settings>
@@
 <text x="92.344" y="115.554" size="1.9304" layer="22" font="vector" rot="MR0" align="center">P1</text>
 <text x="91.836" y="103.292" size="1.9304" layer="21" font="vector" align="center">P2*</text>
-<text x="82.8548" y="39.574725" size="1.9304" layer="22" font="vector" rot="MR0" align="center">HF1R00</text>
+<text x="82.8548" y="39.574725" size="1.9304" layer="22" font="vector" rot="MR0" align="center">HF1R01</text>
 <rectangle x1="82.32266875" y1="40.059103125" x2="82.3374" y2="40.073834375" layer="21"/>
 <rectangle x1="82.204815625" y1="40.073834375" x2="82.352134375" y2="40.088565625" layer="21"/>
@@
 <attribute name="VALUE" x="89.9414" y="83.5914" size="1.27" layer="27" ratio="10" rot="R270"/>
 </element>
+<element name="JP4" library="jumper" library_urn="urn:adsk.eagle:library:252" package="JP1" package3d_urn="urn:adsk.eagle:package:15455/1" value="61300211121" x="75.438" y="81.534" smashed="yes" rot="R180">
+<attribute name="MFN" value="Wurth Electronics Inc." x="75.438" y="81.534" size="1.778" layer="27" rot="R180" display="off"/>
+<attribute name="MPN" value="61300211121" x="75.438" y="81.534" size="1.778" layer="27" rot="R180" display="off"/>
+<attribute name="NAME" x="73.787" y="79.248" size="1.27" layer="25" ratio="10" rot="R90"/>
+<attribute name="OCTOPART_URL" value="https://octopart.com/61300211121-w%C3%BCrth+elektronik-20081794?r=sp&amp;s=_qjp-sYDSLeHQoC-C2Sr3Q" x="75.438" y="81.534" size="1.778" layer="27" rot="R180" display="off"/>
+<attribute name="VALUE" x="72.517" y="84.074" size="1.27" layer="27" ratio="10" rot="R270"/>
+</element>
 </elements>
 <signals>
@@
 <contactref element="P5" pad="PAD_PU12"/>
 <contactref element="P6" pad="PAD_PU12"/>
-<contactref element="SV1" pad="1"/>
-<contactref element="SV1" pad="17"/>
-<contactref element="C2" pad="1"/>
 <contactref element="U1" pad="8"/>
 <contactref element="C3" pad="1"/>
@@
 <contactref element="P5" pad="PAD_PU10"/>
 <contactref element="P5" pad="PAD_PU11"/>
-<wire x1="75.7174" y1="103.1122" x2="76.5886" y2="103.13" width="0.6096" layer="1"/>
-<wire x1="76.5886" y1="103.13" x2="77.723996875" y2="103.13" width="0.6096" layer="1"/>
-<wire x1="77.724" y1="103.13" x2="78.74" y2="103.13" width="0.6096" layer="1"/>
 <wire x1="90.1954" y1="76.9366" x2="91.4518" y2="76.9366" width="0.6096" layer="1"/>
 <wire x1="91.4518" y1="76.9366" x2="91.948" y2="76.4404" width="0.6096" layer="1"/>
 <wire x1="86.233" y1="72.175" x2="89.408" y2="72.175" width="0.6096" layer="1"/>
-<wire x1="77.723996875" y1="103.13" x2="77.724" y2="103.129996875" width="0.6096" layer="1"/>
-<wire x1="77.723996875" y1="103.13" x2="77.724" y2="103.13" width="0.6096" layer="1"/>
-<wire x1="77.724" y1="103.13" x2="78.53425625" y2="103.538290625" width="0.6096" layer="1"/>
-<wire x1="77.724" y1="103.129996875" x2="78.53425625" y2="102.72170625" width="0.6096" layer="1"/>
-<wire x1="78.53425625" y1="102.72170625" x2="78.534259375" y2="102.72170625" width="0.6096" layer="1"/>
-<wire x1="78.74" y1="103.13" x2="78.534259375" y2="102.72170625" width="0.6096" layer="1"/>
-<wire x1="77.724" y1="103.129996875" x2="78.53425625" y2="103.538290625" width="0.6096" layer="1"/>
-<wire x1="78.74" y1="103.13" x2="78.53425625" y2="103.538290625" width="0.6096" layer="1"/>
-<wire x1="77.724" y1="103.13" x2="78.53425625" y2="102.72170625" width="0.6096" layer="1"/>
-<wire x1="78.74" y1="103.13" x2="78.53425625" y2="102.72170625" width="0.6096" layer="1"/>
-<wire x1="77.724" y1="103.13" x2="78.534259375" y2="103.538290625" width="0.6096" layer="1"/>
-<wire x1="78.74" y1="103.13" x2="78.534259375" y2="103.538290625" width="0.6096" layer="1"/>
 <polygon width="0.1016" layer="1" isolate="0.3048" thermals="no">
 <vertex x="74.34026875" y="64.0009375"/>
@@
 <vertex x="65.67970625" y="49.001659375"/>
 </polygon>
+<contactref element="JP4" pad="2"/>
 </signal>
 <signal name="TXD1">
@@
 <contactref element="P2" pad="PAD_PU5"/>
 <contactref element="P5" pad="PAD_PU4"/>
-<wire x1="73.025" y1="86.15" x2="77.133" y2="86.15" width="0.4064" layer="1"/>
-<wire x1="77.133" y1="86.15" x2="77.597" y2="86.614" width="0.4064" layer="1"/>
-<wire x1="77.597" y1="86.614" x2="83.5406" y2="86.614" width="0.4064" layer="1"/>
-<wire x1="83.5406" y1="86.614" x2="84.709" y2="87.7824" width="0.4064" layer="1"/>
-<wire x1="84.709" y1="87.7824" x2="84.709" y2="87.884" width="0.4064" layer="1"/>
 <via x="88.9" y="87.884" extent="1-16" drill="0.4"/>
-<via x="84.709" y="87.884" extent="1-16" drill="0.4"/>
-<wire x1="84.709" y1="87.884" x2="88.9" y2="87.884" width="0.4064" layer="16"/>
-<wire x1="70.61" y1="86.15" x2="73.025" y2="86.15" width="1.27" layer="1"/>
+<via x="75.311" y="87.503" extent="1-16" drill="0.4"/>
+<wire x1="88.519" y1="87.503" x2="88.9" y2="87.884" width="0.4064" layer="16"/>
+<wire x1="73.025" y1="86.15" x2="70.61" y2="86.15" width="1.27" layer="1"/>
 <wire x1="95.39" y1="86.15" x2="93.656" y2="87.884" width="1.27" layer="1"/>
 <wire x1="93.656" y1="87.884" x2="88.9" y2="87.884" width="1.27" layer="1"/>
+<wire x1="75.311" y1="87.503" x2="73.958" y2="86.15" width="0.4064" layer="1"/>
+<wire x1="73.958" y1="86.15" x2="73.025" y2="86.15" width="0.508" layer="1"/>
+<wire x1="75.311" y1="87.503" x2="76.962" y2="89.154" width="0.4064" layer="16"/>
+<wire x1="76.962" y1="89.154" x2="82.55" y2="89.154" width="0.4064" layer="16"/>
+<wire x1="84.201" y1="87.503" x2="88.519" y2="87.503" width="0.4064" layer="16"/>
+<wire x1="82.55" y1="89.154" x2="84.201" y2="87.503" width="0.4064" layer="16"/>
 </signal>
 <signal name="RXD4">
@@
 <contactref element="P2" pad="PAD_PD5"/>
 <contactref element="P5" pad="PAD_PD4"/>
-<wire x1="73.787" y1="86.15" x2="77.133" y2="86.15" width="0.4064" layer="16"/>
-<wire x1="77.133" y1="86.15" x2="77.597" y2="86.614" width="0.4064" layer="16"/>
+<wire x1="77.597" y1="86.614" x2="77.133" y2="86.15" width="0.4064" layer="16"/>
 <wire x1="77.597" y1="86.614" x2="82.607" y2="86.614" width="0.4064" layer="16"/>
 <wire x1="82.607" y1="86.614" x2="83.071" y2="86.15" width="0.4064" layer="16"/>
@@
 <wire x1="95.39" y1="86.15" x2="91.992" y2="86.15" width="1.27" layer="16"/>
 <wire x1="91.992" y1="86.15" x2="91.948" y2="86.106" width="1.27" layer="16"/>
-<wire x1="70.61" y1="86.15" x2="73.787" y2="86.15" width="1.27" layer="16"/>
+<wire x1="73.787" y1="86.15" x2="70.61" y2="86.15" width="1.27" layer="16"/>
+<wire x1="77.133" y1="86.15" x2="73.787" y2="86.15" width="0.4064" layer="16"/>
 </signal>
 <signal name="TXD6">
@@
 <wire x1="70.61" y1="56.15" x2="73.166" y2="53.594" width="1.27" layer="1"/>
 <wire x1="88.011" y1="53.594" x2="92.837" y2="53.594" width="0.4064" layer="16"/>
-<wire x1="92.837" y1="53.594" x2="95.376075" y2="56.133075" width="1.27" layer="1"/>
-<wire x1="95.376075" y1="56.133075" x2="95.376075" y2="56.1419625" width="1.27" layer="1"/>
-<wire x1="95.376075" y1="56.133075" x2="95.39" y2="56.15" width="0" layer="19" extent="1-1"/>
+<wire x1="95.39" y1="56.15" x2="92.837" y2="53.597" width="1.27" layer="1"/>
+<wire x1="92.837" y1="53.597" x2="92.837" y2="53.594" width="1.27" layer="1"/>
 </signal>
 <signal name="RXD5">
@@
 <wire x1="88.9254" y1="78.2574" x2="88.9254" y2="76.9366" width="0.6096" layer="1"/>
 </signal>
+<signal name="N$3">
+<contactref element="SV1" pad="1"/>
+<contactref element="SV1" pad="17"/>
+<contactref element="C2" pad="1"/>
+<wire x1="75.7174" y1="103.1122" x2="76.5886" y2="103.13" width="0.6096" layer="1"/>
+<wire x1="76.5886" y1="103.13" x2="77.723996875" y2="103.13" width="0.6096" layer="1"/>
+<wire x1="77.724" y1="103.13" x2="78.74" y2="103.13" width="0.6096" layer="1"/>
+<wire x1="77.723996875" y1="103.13" x2="77.724" y2="103.129996875" width="0.6096" layer="1"/>
+<wire x1="77.723996875" y1="103.13" x2="77.724" y2="103.13" width="0.6096" layer="1"/>
+<wire x1="77.724" y1="103.13" x2="78.53425625" y2="103.538290625" width="0.6096" layer="1"/>
+<wire x1="77.724" y1="103.129996875" x2="78.53425625" y2="102.72170625" width="0.6096" layer="1"/>
+<wire x1="78.53425625" y1="102.72170625" x2="78.534259375" y2="102.72170625" width="0.6096" layer="1"/>
+<wire x1="78.74" y1="103.13" x2="78.534259375" y2="102.72170625" width="0.6096" layer="1"/>
+<wire x1="77.724" y1="103.129996875" x2="78.53425625" y2="103.538290625" width="0.6096" layer="1"/>
+<wire x1="78.74" y1="103.13" x2="78.53425625" y2="103.538290625" width="0.6096" layer="1"/>
+<wire x1="77.724" y1="103.13" x2="78.53425625" y2="102.72170625" width="0.6096" layer="1"/>
+<wire x1="78.74" y1="103.13" x2="78.53425625" y2="102.72170625" width="0.6096" layer="1"/>
+<wire x1="77.724" y1="103.13" x2="78.534259375" y2="103.538290625" width="0.6096" layer="1"/>
+<wire x1="78.74" y1="103.13" x2="78.534259375" y2="103.538290625" width="0.6096" layer="1"/>
+<contactref element="JP4" pad="1"/>
+<wire x1="78.74" y1="82.81" x2="78.734" y2="82.804" width="0.3048" layer="1"/>
+<wire x1="78.734" y1="82.804" x2="75.438" y2="82.804" width="0.508" layer="1"/>
+<wire x1="75.438" y1="82.804" x2="76.962" y2="84.328" width="0.4064" layer="1"/>
+<wire x1="75.7174" y1="101.3206" x2="75.7174" y2="103.1122" width="0.4064" layer="1"/>
+<wire x1="76.962" y1="84.328" x2="76.962" y2="100.076" width="0.4064" layer="1"/>
+<wire x1="76.962" y1="100.076" x2="75.7174" y2="101.3206" width="0.4064" layer="1"/>
+</signal>
 </signals>
